File: Teensy_Daughtercard/Teensy_Daughtercard.kicad_sch (KiCad schematic)
At the start: 15 parts, among them J1 XG4A-5034, J2 Conn_01x24_Socket, J3 Conn_01x24_Socket, J4 Conn_01x24_Pin, J5 Conn_01x24_Pin, J6 LPJ4012AHNL, U1 Teensy4.1

Commit message: First draft complete
Parts:
- removed H1, H4: MH, MountingHole:MountingHole_3.5mm_Pad, symbol Mechanical:MountingHole_Pad
- renumbered H2 to H1, H3 to H2, J6 to J1, J4 to J3, J3 to J4, J1 to J6
Connections:
- net DIR1: now also U1.24 (32_OUT1B); no longer U1.3 (1_TX1_CTX2_MISO1)
- net DIR2: now also U1.33 (41_A17); no longer U1.19 (27_A13_SCK1)
- net DIR3: now also U1.30 (38_CS1_IN1); no longer U1.44 (22_A8_CTX1)
- net DIR4: now also U1.25 (33_MCLK2); no longer U1.22 (30_CRX3)
- net ENA1: now also U1.27 (35_TX8); no longer U1.23 (31_CTX3)
- net ENA2: now also U1.37 (15_A1_RX3_SPDIF_IN); no longer U1.42 (20_A6_TX5_LRCLK1)
- net ENA3: now also U1.31 (39_MISO1_OUT1A); no longer U1.20 (28_RX7)
- net ENA4: now also U1.28 (36_CS); no longer U1.45 (23_A9_CRX1_MCLK1)
- net GPIO1: now also U1.2 (0_RX1_CRX2_CS1); no longer U1.37 (15_A1_RX3_SPDIF_IN)
- net GPIO2: now also U1.4 (2_OUT2); no longer U1.10 (8_TX2_IN1)
- net GPIO3: now also U1.6 (4_BCLK2); no longer U1.11 (9_OUT1C)
- net GPIO4: now also U1.8 (6_OUT1D); no longer U1.9 (7_RX2_OUT1A)
- net Imon PS1: now also U1.45 (23_A9_CRX1_MCLK1); no longer U1.17 (25_A11_RX6_SDA2)
- net Imon PS2: now also U1.44 (22_A8_CTX1); no longer U1.16 (24_A10_TX6_SCL2)
- net PUL1: now also U1.26 (34_RX8); no longer U1.2 (0_RX1_CRX2_CS1)
- net PUL2: now also U1.36 (14_A0_TX3_SPDIF_OUT); no longer U1.18 (26_A12_MOSI1)
- net PUL3: now also U1.32 (40_A16); no longer U1.43 (21_A7_RX5_BCLK1)
- net PUL4: now also U1.29 (37_CS); no longer U1.21 (29_TX7)
- net RELAY1: now also U1.23 (31_CTX3); no longer U1.24 (32_OUT1B)
- net RELAY10: now also U1.10 (8_TX2_IN1); no longer U1.8 (6_OUT1D)
- net RELAY11: now also U1.9 (7_RX2_OUT1A); no longer U1.29 (37_CS)
- net RELAY12: now also U1.7 (5_IN2); no longer U1.30 (38_CS1_IN1)
- net RELAY13: now also U1.5 (3_LRCLK2); no longer U1.31 (39_MISO1_OUT1A)
- net RELAY14: now also U1.3 (1_TX1_CTX2_MISO1); no longer U1.32 (40_A16)
- net RELAY15: now also U1.43 (21_A7_RX5_BCLK1); no longer U1.36 (14_A0_TX3_SPDIF_OUT)
- net RELAY16: now also U1.42 (20_A6_TX5_LRCLK1); no longer U1.33 (41_A17)
- net RELAY2: now also U1.22 (30_CRX3); no longer U1.4 (2_OUT2)
- net RELAY3: now also U1.21 (29_TX7); no longer U1.25 (33_MCLK2)
- net RELAY4: now also U1.20 (28_RX7); no longer U1.5 (3_LRCLK2)
- net RELAY5: now also U1.19 (27_A13_SCK1); no longer U1.26 (34_RX8)
- net RELAY6: now also U1.18 (26_A12_MOSI1); no longer U1.6 (4_BCLK2)
- net RELAY7: now also U1.16 (24_A10_TX6_SCL2); no longer U1.7 (5_IN2)
- net RELAY8: now also U1.17 (25_A11_RX6_SDA2); no longer U1.27 (35_TX8)
- net RELAY9: now also U1.11 (9_OUT1C); no longer U1.28 (36_CS)
- net SCLTC: now also U1.41 (19_A5_SCL); no longer U1.40 (18_A4_SDA)
- net SDATC: now also U1.40 (18_A4_SDA); no longer U1.41 (19_A5_SCL)
Other:
- note added: "TODO: Add Power LED Design Reviews"
- note removed: "TODO: Line up the connectors with the Teensy and redo the PCB layout"
- moved on the sheet: H2

Commit message: First revision 6/11
Parts:
- added LED1: LTST-C190YKT, LIST-C190YKT:LEDC1608X90N, symbol LTST-C190YKT:LTST-C190YKT
- added R1: 500, Resistor_SMD:R_0805_2012Metric_Pad1.20x1.40mm_HandSolder, symbol Device:R
Connections:
- net GNDD: now also LED1.1 (K)
- net VMC+: now also R1.2
- new net: LED1.2 (A), R1.1

Commit message: Replaced Magjack
Parts:
- removed J1: LPJ4012AHNL, LPJ4012AHNL:LPJ4012AHNL, symbol LPJ4012AHNL:LPJ4012AHNL
- added J1: 1664073, 1664073:1664073, symbol 1664073:1664073
Connections:
- net ETH_LED: now also J1.P11 (A_GREEN)
- net ETH_RX+: now also J1.P4 (RD+)
- net ETH_RX-: now also J1.P6 (RD-)
- net ETH_TX+: now also J1.P1 (TD+)
- net ETH_TX-: now also J1.P3 (TD-)
- net GNDD: now also J1.P12 (K_GREEN), J1.P8 (CHS_GROUND)
- net at C1.2: now also J1.P2 (TCT), J1.P5 (RCT)
- no-connect marks 115 -> 116

Commit message: Final changes
Parts:
- R1: value 500 -> 1000
- renumbered J4 to J3, J3 to J4
Other:
- moved on the sheet: J3, J4
